File: switch_network.kicad_sch (KiCad schematic)
At the start: 140 parts, among them SW10 MX_SW_HS, SW11 MX_SW_HS, SW12 MX_SW_HS, SW13 MX_SW_HS, SW14 MX_SW_HS, SW15 MX_SW_HS, SW16 MX_SW_HS, SW17 MX_SW_HS, SW18 MX_SW_HS, SW19 MX_SW_HS, SW20 MX_SW_HS, SW21 MX_SW_HS, SW22 MX_SW_HS, SW23 MX_SW_HS, SW24 MX_SW_HS, SW25 MX_SW_HS, SW26 MX_SW_HS, SW27 MX_SW_HS, SW28 MX_SW_HS, SW29 MX_SW_HS, SW30 MX_SW_HS, SW31 MX_SW_HS, SW32 MX_SW_HS, SW33 MX_SW_HS, SW34 MX_SW_HS, SW35 MX_SW_HS, SW36 MX_SW_HS, SW37 MX_SW_HS, SW38 MX_SW_HS, SW39 MX_SW_HS, SW4 MX_SW_HS, SW40 MX_SW_HS, SW41 MX_SW_HS, SW42 MX_SW_HS, SW43 MX_SW_HS, SW44 MX_SW_HS, SW45 MX_SW_HS, SW46 MX_SW_HS, SW47 MX_SW_HS, SW48 MX_SW_HS, SW49 MX_SW_HS, SW5 MX_SW_HS, SW50 MX_SW_HS, SW51 MX_SW_HS, SW52 MX_SW_HS, SW53 MX_SW_HS, SW54 MX_SW_HS, SW55 MX_SW_HS, SW56 MX_SW_HS, SW57 MX_SW_HS, SW58 MX_SW_HS, SW59 MX_SW_HS, SW6 MX_SW_HS, SW60 MX_SW_HS, SW61 MX_SW_HS, SW62 MX_SW_HS, SW63 MX_SW_HS, SW64 MX_SW_HS, SW65 MX_SW_HS, SW66 MX_SW_HS, SW67 MX_SW_HS, SW68 MX_SW_HS, SW69 MX_SW_HS, SW7 MX_SW_HS, SW70 MX_SW_HS, SW71 MX_SW_HS, SW8 MX_SW_HS, SW9 MX_SW_HS

Commit message: code?
Parts:
- SW10, SW11, SW12, SW13, SW14, SW15, SW16, SW17, SW18, SW20, SW21, SW22, SW23, SW24, SW25, SW26, SW27, SW28, SW29, SW30, SW31, SW33, SW35, SW36, SW37, SW38, SW39, SW4, SW40, SW41, SW42, SW43, SW44, SW45, SW46, SW47, SW48, SW49, SW5, SW50, SW51, SW52, SW53, SW54, SW55, SW56, SW57, SW58, SW6, SW7, SW8, SW9: footprint marbastmx:SW_MX_HS_1u -> marbastmx:SW_MX_1u
- SW19, SW32: footprint marbastmx:SW_MX_HS_1.5u -> marbastmx:SW_MX_1.5u
- SW34: footprint marbastmx:SW_MX_HS_1.75u -> marbastmx:SW_MX_1.75u
- SW59: renamed from SW60; footprint marbastmx:SW_MX_HS_1.75u -> marbastmx:SW_MX_1.75u
- SW60: renamed from SW61; footprint marbastmx:SW_MX_HS_1u -> marbastmx:SW_MX_1u
- SW61: renamed from SW62; footprint marbastmx:SW_MX_HS_1u -> marbastmx:SW_MX_1u
- SW62: renamed from SW63; footprint marbastmx:SW_MX_HS_1.25u -> marbastmx:SW_MX_1.25u
- SW63: renamed from SW64; footprint marbastmx:SW_MX_HS_1.25u -> marbastmx:SW_MX_1.25u
- SW64: renamed from SW65; footprint marbastmx:SW_MX_HS_1.25u -> marbastmx:SW_MX_1.25u
- SW65: renamed from SW66; footprint marbastmx:SW_MX_HS_1u -> marbastmx:SW_MX_1u
- SW66: renamed from SW67; footprint marbastmx:SW_MX_HS_1u -> marbastmx:SW_MX_1u
- SW67: renamed from SW68; footprint marbastmx:SW_MX_HS_1u -> marbastmx:SW_MX_1u
- SW68: renamed from SW69; footprint marbastmx:SW_MX_HS_1u -> marbastmx:SW_MX_1u
- SW69: renamed from SW70; footprint marbastmx:SW_MX_HS_1u -> marbastmx:SW_MX_1u
- SW70: renamed from SW71; footprint marbastmx:SW_MX_HS_1u -> marbastmx:SW_MX_1u
- SW71: renamed from SW59; footprint marbastmx:SW_MX_HS_1u -> marbastmx:SW_MX_1u
- renumbered D9 to D10, D10 to D11, D11 to D12, D12 to D13, D13 to D14, D14 to D15, D15 to D16, D16 to D17, D17 to D18, D18 to D19, D1 to D2, D19 to D20, D20 to D21, D21 to D22, D22 to D23, D23 to D24, D24 to D25, D25 to D26, D26 to D27, D27 to D28, D28 to D29, D2 to D3, D29 to D30, D30 to D31, D31 to D32, D32 to D33, D33 to D34, D34 to D35, D35 to D36, D36 to D37, D37 to D38, D38 to D39, D3 to D4, D39 to D40, D40 to D41, D41 to D42, D42 to D43, D43 to D44, D44 to D45, D45 to D46, D46 to D47, D47 to D48, D48 to D49, D4 to D5, D49 to D50, D50 to D51, D51 to D52, D52 to D53, D53 to D54, D54 to D55, D55 to D56, D5 to D6, D56 to D69, D6 to D7, D7 to D8, D8 to D9
Connections:
- no-connect marks 1 -> 0
